Commit message: v2.0

File: src/dog_bringup/urdf/const.xacro (robot description, xacro)
@@ -39,5 +39,5 @@
 <xacro:property name="shank_izz" value="0.000031266"/>    <!-- 小腿绕z轴转动惯量(kg·m²) -->
 <!-- 脚部参数 -->
-<xacro:property name="foot_mass" value="0.02"/>           <!-- 脚部质量(kg) -->
+<xacro:property name="foot_mass" value="0.06"/>           <!-- 脚部质量(kg) -->
 <xacro:property name="foot_radius" value="0.023"/>        <!-- 脚部半径(m) -->
 <xacro:property name="foot_ixx" value="0.0001"/>          <!-- 脚部绕x轴转动惯量(kg·m²) -->

File: src/dog_bringup/urdf/leg.xacro (robot description, xacro)
@@ -106,11 +106,30 @@
             <preserveFixedJoint>true</preserveFixedJoint>
         </gazebo>
+        <gazebo reference="${name}_HIP">
+            <mu1>0.2</mu1>
+            <mu2>0.2</mu2>
+            <material>Gazebo/Yellow</material>
+            <self_collide>1</self_collide>
+        </gazebo>
+        <gazebo reference="${name}_THIGH">
+            <mu1>0.2</mu1>
+            <mu2>0.2</mu2>
+            <material>Gazebo/Blue</material>
+            <self_collide>0</self_collide>
+            <kp value="1000000.0"/>
+            <kd value="100.0"/>
+        </gazebo>
+        <gazebo reference="${name}_SHANK">
+            <mu1>0.6</mu1>
+            <mu2>0.6</mu2>
+            <material>Gazebo/DarkGrey</material>
+            <self_collide>1</self_collide>
+        </gazebo>
         <gazebo reference="${name}_FOOT">
-            <mu1>1.5</mu1>
-            <mu2>1.5</mu2>
+            <mu1>1.0</mu1>
+            <mu2>1.0</mu2>
             <kp>1000000.0</kp>
-            <kd>100.0</kd>
-            <maxVel>0.0</maxVel>
-            <minDepth>0.001</minDepth>
+            <kd>10000.0</kd>
+            <self_collide>1</self_collide>
             <sensor name="${name}_contact_sensor" type="contact">
               <always_on>true</always_on>
