Commit message: 修改了小腿装反的bug，优化了小腿转动逻辑

File: leg_control/src/leg_model_1/urdf/leg_model_1.urdf (robot description, URDF)
Before this commit: robot leg_model_1, 6 links, 5 joints
Joints:
- joint Knee_joint: limit lower=-21 upper=21 effort=20 velocity=20 -> lower=-3.14 upper=3.14 effort=20 velocity=20; mimic joint=thigh_joint multiplier=6.666667 offset=2 -> joint=thigh_joint multiplier=1 offset=0.5
- joint thigh_joint: limit lower=-0.55 upper=0.15 effort=20 velocity=20 -> lower=-3.14 upper=3.14 effort=20 velocity=20; origin xyz=0 0 -0.0823 rpy=-3.1416 0 0 -> xyz=0 0 -0.0823 rpy=0 0 3.1416
