Commit message: 添加了步态控制算法，完善了小腿运动的不足

File: leg_control/src/leg_model/urdf/leg_model.urdf (robot description, URDF)
Before this commit: robot leg_model, 8 links, 7 joints
Joints:
- joint knee_crank_joint: limit lower=-3.14 upper=3.14 effort=20 velocity=20 -> lower=-0.80 upper=1.20 effort=20 velocity=20
