Commit message: 存档

File: src/dog_bringup/xacro/cdut_dog/dog.xacro (robot description, xacro)
@@ -43,4 +43,64 @@
         <origin xyz="0 0 0" rpy="0 0 0"/>
     </joint>
+    <!-- 仿真用前向 2D 雷达，输出 PointCloud2 到 /points。 -->
+    <link name="lidar_link">
+        <inertial>
+            <mass value="0.05"/>
+            <origin xyz="0 0 0" rpy="0 0 0"/>
+            <inertia ixx="0.00002" ixy="0.0" ixz="0.0" iyy="0.00002" iyz="0.0" izz="0.00002"/>
+        </inertial>
+        <visual>
+            <geometry>
+                <cylinder radius="0.025" length="0.035"/>
+            </geometry>
+            <material name="lidar_black">
+                <color rgba="0.02 0.02 0.02 1.0"/>
+            </material>
+        </visual>
+        <collision>
+            <geometry>
+                <cylinder radius="0.025" length="0.035"/>
+            </geometry>
+        </collision>
+    </link>
+    <joint name="lidar_joint" type="fixed">
+        <parent link="TORSO"/>
+        <child link="lidar_link"/>
+        <origin xyz="0.22 0 0.01" rpy="0 0 0"/>
+    </joint>
+    <gazebo reference="lidar_link">
+      <sensor name="front_lidar" type="ray">
+        <always_on>true</always_on>
+        <visualize>true</visualize>
+        <update_rate>15</update_rate>
+        <ray>
+          <scan>
+            <horizontal>
+              <samples>181</samples>
+              <resolution>1</resolution>
+              <min_angle>-1.0472</min_angle>
+              <max_angle>1.0472</max_angle>
+            </horizontal>
+          </scan>
+          <range>
+            <min>0.12</min>
+            <max>5.0</max>
+            <resolution>0.01</resolution>
+          </range>
+          <noise>
+            <type>gaussian</type>
+            <mean>0.0</mean>
+            <stddev>0.01</stddev>
+          </noise>
+        </ray>
+        <plugin name="front_lidar_points" filename="libgazebo_ros_ray_sensor.so">
+          <ros>
+            <remapping>~/out:=/points</remapping>
+          </ros>
+          <output_type>sensor_msgs/PointCloud2</output_type>
+          <frame_name>lidar_link</frame_name>
+        </plugin>
+      </sensor>
+    </gazebo>
     <xacro:dog_leg name="LF" mirror="1" f_b="1"/>
     <xacro:dog_leg name="LH" mirror="1" f_b="-1"/>
